Commit message: Created core URDF (robot_core.xacro)

File: description/robot.urdf.xacro (robot description, xacro)
@@ -1,4 +1,4 @@
 <?xml version="1.0"?>
 <robot xmlns:xacro="http://www.ros.org/wiki/xacro"  name="robot">
-    <xacro:include filename="robot_core.xacro" />
+    <xacro:include filename="robot_core.xacro"/>
 </robot>

File: description/robot_core.xacro (robot description, xacro)
@@ -1,3 +1,157 @@
 <?xml version="1.0"?>
 <robot xmlns:xacro="http://www.ros.org/wiki/xacro" >
+    <xacro:include filename="inertial_macros.xacro"/>
+    <!-- colors -->
+    <material name="blue">
+        <color rgba="0 0 1 1"/>
+    </material>
+    <material name="grey">
+        <color rgba="1 1 1 1"/>
+    </material>
+    <material name="light_grey">
+        <color rgba="0.5 0.5 0.5 0.5"/>
+    </material>
+    <material name="black">
+        <color rgba="0 0 0 1"/>
+    </material>
+    <!-- Base Link-->
+    <link name="base_link">
+    </link>
+    <!-- Chassis-->
+    <joint name="chassis_joint" type="fixed">
+        <parent link="base_link"/>
+        <child link="chassis"/>
+        <origin xyz="-0.1 0 0"/>
+    </joint>
+    <link name="chassis">
+        <visual>
+            <origin xyz="0.55245 0 0.4572"/>
+            <geometry>
+                <box size="1.1049 0.6096 0.9144"/>
+            </geometry>
+            <material name="grey"/>
+        </visual>
+        <collision>
+            <origin xyz="0.55245 0 0.4572"/>
+            <geometry>
+                <box size="1.1049 0.6096 0.9144"/>
+            </geometry>
+        </collision>
+        <xacro:inertial_box mass="0.5" x="1.1049" y="0.6096" z="0.9144">
+            <origin xyz="0.55245 0 0.4572" rpy="0 0 0"/>
+        </xacro:inertial_box>
+    </link>
+    <!-- <gazebo reference="chassis">
+        <material>Gazebo/White</material>
+    </gazebo> -->
+    <!-- LEFT WHEEL LINK -->
+    <joint name="left_wheel_joint" type="continuous">
+        <parent link="base_link"/>
+        <child link="left_wheel"/>
+        <origin xyz="0 0.3248 0.2032" rpy="-${pi/2} 0 0" />
+        <axis xyz="0 0 1"/>
+    </joint>
+    <link name="left_wheel">
+        <visual>
+            <!-- <origin xyz="0 -0.2032 0"/> -->
+            <geometry>
+                <cylinder radius="0.3048" length="0.04"/>
+            </geometry>
+            <material name="black"/>
+        </visual>
+        <collision>
+            <geometry>
+                <cylinder radius="0.3048" length="0.04"/>
+            </geometry>
+        </collision>
+        <xacro:inertial_cylinder mass="0.1" length="0.04" radius="0.3048">
+            <origin xyz="0 0 0" rpy="0 0 0"/>
+        </xacro:inertial_cylinder>
+    </link>
+    <!-- <gazebo reference="left_wheel">
+        <material>Gazebo/Blue</material>
+    </gazebo> -->
+    <!-- RIGHT WHEEL LINK -->
+    <joint name="right_wheel_joint" type="continuous">
+        <parent link="base_link"/>
+        <child link="right_wheel"/>
+        <origin xyz="0 -0.3248 0.2032" rpy="${pi/2} 0 0" />
+        <axis xyz="0 0 -1"/>
+    </joint>
+    <link name="right_wheel">
+        <visual>
+            <!-- <origin xyz="0 0.2032 0"/> -->
+            <geometry>
+                <cylinder radius="0.3048" length="0.04"/>
+            </geometry>
+            <material name="black"/>
+        </visual>
+        <collision>
+            <geometry>
+                <cylinder radius="0.3048" length="0.04"/>
+            </geometry>
+        </collision>
+        <xacro:inertial_cylinder mass="0.1" length="0.04" radius="0.3048">
+            <origin xyz="0 0 0" rpy="0 0 0"/>
+        </xacro:inertial_cylinder>
+    </link>
+    <!-- <gazebo reference="right_wheel">
+        <material>Gazebo/Blue</material>
+    </gazebo> -->
+    <!-- CASTER LEFT WHEEL LINK -->
+    <joint name="caster_left_wheel_joint" type="continuous">
+        <parent link="chassis"/>
+        <child link="caster_left_wheel"/>
+        <origin xyz="1.1049 0.3148 0" rpy="${pi/2} 0 0" />
+        <axis xyz="0 0 -1"/>
+    </joint>
+    <link name="caster_left_wheel">
+        <visual>
+            <geometry>
+                <cylinder radius="0.1016" length="0.02"/>
+            </geometry>
+            <material name="black"/>
+        </visual>
+        <collision>
+            <geometry>
+                <cylinder radius="0.1016" length="0.2"/>
+            </geometry>
+        </collision>
+        <xacro:inertial_sphere mass="0.1" radius="0.1016">
+            <origin xyz="0 0 0" rpy="0 0 0"/>
+        </xacro:inertial_sphere>
+    </link>
+    <!-- <gazebo reference="caster_left_wheel">
+        <material>Gazebo/Black</material>
+        <mu1 value="0.001"/>
+        <mu2 value="0.001"/>
+    </gazebo> -->
+    <!-- CASTER RIGHT WHEEL LINK -->
+    <joint name="caster_right_wheel_joint" type="continuous">
+        <parent link="chassis"/>
+        <child link="caster_right_wheel"/>
+        <origin xyz="1.1049 -0.3148 0" rpy="${pi/2} 0 0" />
+        <axis xyz="0 0 -1"/>
+    </joint>
+    <link name="caster_right_wheel">
+        <visual>
+            <geometry>
+                <cylinder radius="0.1016" length="0.02"/>
+            </geometry>
+            <material name="black"/>
+        </visual>
+        <collision>
+            <geometry>
+                <cylinder radius="0.1016" length="0.2"/>
+            </geometry>
+        </collision>
+        <xacro:inertial_sphere mass="0.1" radius="0.1016">
+            <origin xyz="0 0 0" rpy="0 0 0"/>
+        </xacro:inertial_sphere>
+    </link>
+    <!-- <gazebo reference="caster_wheel">
+        <material>Gazebo/Black</material>
+        <mu1 value="0.001"/>
+        <mu2 value="0.001"/>
+    </gazebo> -->
 </robot>
