Commit message: Setup gazebo simulation environment with lidar

File: description/robot.urdf.xacro (robot description, xacro)
@@ -1,5 +1,4 @@
 <?xml version="1.0"?>
-<robot xmlns:xacro="http://www.ros.org/wiki/xacro"  name="robot">
+<robot name="wheelchair" xmlns:xacro="http://www.ros.org/wiki/xacro">
     <xacro:include filename="robot_core.xacro"/>
-    <xacro:include filename="gazebo_control.xacro"/>
 </robot>

File: description/robot_core.xacro (robot description, xacro)
@@ -1,5 +1,74 @@
 <?xml version="1.0"?>
 <robot xmlns:xacro="http://www.ros.org/wiki/xacro" >
-    <xacro:include filename="inertial_macros.xacro"/>
+    <!-- ############################################################## -->
+    <!--                        Geometry & Constants                    -->
+    <!-- ############################################################## -->
+    <!-- Pi Constant -->
+    <xacro:property name="pi_const" value="3.14159265" />
+    <!-- Body Dimensions -->
+    <xacro:property name="l" value="1.1049"/>
+    <xacro:property name="w" value="0.6096"/>
+    <xacro:property name="h" value="0.6144"/>   <!-- actual: 0.9144-->
+    <!-- Wheel Dimension -->
+    <xacro:property name="r_wheel" value="0.3048"/>
+    <xacro:property name="t_wheel" value="0.0400"/>
+    <!-- Caster Dimension -->
+    <xacro:property name="r_caster" value="0.1016"/>
+    <xacro:property name="t_caster" value="0.0200"/>
+    <!-- Distance btw Centers -->
+    <xacro:property name="body_to_gnd" value="${h/2+r_caster}"/>
+    <xacro:property name="wheel_to_body_side" value="0.55245"/>
+    <xacro:property name="caster_to_body_side" value="0.14605"/>
+    <xacro:property name="wheel_to_body_top" value="${w/2+t_wheel/2}"/>
+    <xacro:property name="caster_to_body_top" value="${w/2+t_caster/2}"/>
+    <!-- Material Density -->
+    <xacro:property name="d_body" value="7850.0"/>
+    <xacro:property name="d_wheel" value="7850.0"/>
+    <xacro:property name="d_caster" value="7850.0"/>
+    <!-- Wheelchair Mass -->
+    <xacro:property name="m_body" value="${d_body*l*w*h}"/>
+    <xacro:property name="m_wheel" value="${d_wheel*pi_const*r_wheel*r_wheel*t_wheel}"/>
+    <xacro:property name="m_caster" value="${d_caster*pi_const*r_caster*r_caster*t_caster}"/>
+    <!-- Moment of Inertia of Body -->
+    <xacro:property name="Ix_body" value="${(1/12)*m_body*(h*h+w*w)}"/>
+    <xacro:property name="Iy_body" value="${(1/12)*m_body*(l*l+h*h)}"/>
+    <xacro:property name="Iz_body" value="${(1/12)*m_body*(l*l+w*w)}"/>
+    <!-- Moment of Inertia of Wheel -->
+    <xacro:property name="I_wheel" value="${(1.0/12.0)*m_wheel*(3.0*r_wheel*r_wheel+t_wheel*t_wheel)}"/>
+    <xacro:property name="Iz_wheel" value="${0.5*m_wheel*r_wheel*r_wheel}"/>
+    <!-- Moment of Inertia of Caster -->
+    <xacro:property name="I_caster" value="${(1.0/12.0)*m_caster*(3.0*r_caster*r_caster+t_caster*t_caster)}"/>
+    <xacro:property name="Iz_caster" value="${0.5*m_caster*r_caster*r_caster}"/>
+    <!-- Macro for Inertial Section -->
+    <xacro:macro name="inertia_body">
+        <!-- displacement & rientation of center of mass frame of link to ground -->
+        <inertial>
+            <origin xyz="0 0 ${body_to_gnd}" rpy="0 0 0"/>
+            <mass value="${m_body}"/>
+            <inertia ixx="${Ix_body}" ixy="0.0" ixz="0.0"
+                     iyy="${Iy_body}" iyz="0.0"
+                     izz="${Iz_body}"/>
+        </inertial>
+    </xacro:macro>
+    <xacro:macro name="inertia_wheel">
+        <inertial>
+            <origin xyz="0 0 0" rpy="${pi_const/2} 0 0"/>
+            <mass value="${m_wheel}"/>
+            <inertia ixx="${I_wheel}" ixy="0.0" ixz="0.0"
+                     iyy="${I_wheel}" iyz="0.0"
+                     izz="${Iz_wheel}"/>
+        </inertial>
+    </xacro:macro>
+    <xacro:macro name="inertia_caster">
+        <inertial>
+            <origin xyz="0 0 0" rpy="${pi_const/2} 0 0"/>
+            <mass value="${m_caster}"/>
+            <inertia ixx="${I_caster}" ixy="0.0" ixz="0.0"
+                     iyy="${I_caster}" iyz="0.0"
+                     izz="${Iz_caster}"/>
+        </inertial>
+    </xacro:macro>
+    <!-- Additional Files -->
+    <xacro:include filename="$(find wheelchair_one)/description/gazebo_control"/>
     <!-- colors -->
     <material name="blue">
@@ -15,143 +84,158 @@
         <color rgba="0 0 0 1"/>
     </material>
+    <!-- ############################################################## -->
+    <!--                            Links & Joints                      -->
+    <!-- ############################################################## -->
     <!-- Base Link-->
-    <link name="base_link">
-    </link>
+    <link name="base_link"></link>
     <!-- Chassis-->
     <joint name="chassis_joint" type="fixed">
         <parent link="base_link"/>
         <child link="chassis"/>
-        <origin xyz="-0.1 0 0"/>
     </joint>
     <link name="chassis">
         <visual>
-            <origin xyz="0.55245 0 0.4572"/>
-            <geometry>
-                <box size="1.1049 0.6096 0.9144"/>
+            <origin xyz="0 0 ${body_to_gnd}" rpy="0 0 0"/>
+            <geometry>
+                <box size="${l} ${w} ${h}"/>
             </geometry>
             <material name="grey"/>
         </visual>
         <collision>
-            <origin xyz="0.55245 0 0.4572"/>
-            <geometry>
-                <box size="1.1049 0.6096 0.9144"/>
-            </geometry>
-        </collision>
-        <xacro:inertial_box mass="0.5" x="1.1049" y="0.6096" z="0.9144">
-            <origin xyz="0.55245 0 0.4572" rpy="0 0 0"/>
-        </xacro:inertial_box>
-    </link>
-    <gazebo reference="chassis">
-        <material>Gazebo/Grey</material>
-    </gazebo>
+            <origin xyz="0 0 ${body_to_gnd}" rpy="0 0 0"/>
+            <geometry>
+                <box size="${l} ${w} ${h}"/>
+            </geometry>
+        </collision>
+        <xacro:inertia_body/>
+    </link>
     <!-- LEFT WHEEL LINK -->
     <joint name="left_wheel_joint" type="continuous">
-        <parent link="base_link"/>
+        <parent link="chassis"/>
         <child link="left_wheel"/>
-        <origin xyz="0 0.3248 0.2032" rpy="-${pi/2} 0 0" />
-        <axis xyz="0 0 1"/>
+        <origin xyz="${-wheel_to_body_side} ${-wheel_to_body_top} ${r_wheel}" rpy="0 0 0" />
+        <axis xyz="0 1 0"/>
+        <limit effort="50000" velocity="10"/>
+        <dynamic damping="1.0" friction="1.0"/>
     </joint>
     <link name="left_wheel">
         <visual>
-            <!-- <origin xyz="0 -0.2032 0"/> -->
-            <geometry>
-                <cylinder radius="0.3048" length="0.04"/>
+            <origin xyz="0 0 0" rpy="${pi_const/2} 0 0"/>
+            <geometry>
+                <cylinder radius="${r_wheel}" length="${t_wheel}"/>
             </geometry>
             <material name="black"/>
         </visual>
         <collision>
-            <geometry>
-                <cylinder radius="0.3048" length="0.04"/>
-            </geometry>
-        </collision>
-        <xacro:inertial_cylinder mass="0.1" length="0.04" radius="0.3048">
-            <origin xyz="0 0 0" rpy="0 0 0"/>
-        </xacro:inertial_cylinder>
-    </link>
-    <gazebo reference="left_wheel">
-        <material>Gazebo/Black</material>
-    </gazebo>
+            <origin xyz="0 0 0" rpy="${pi_const/2} 0 0"/>
+            <geometry>
+                <cylinder radius="${r_wheel}" length="${t_wheel}"/>
+            </geometry>
+        </collision>
+        <xacro:inertia_wheel/>
+    </link>
     <!-- RIGHT WHEEL LINK -->
     <joint name="right_wheel_joint" type="continuous">
-        <parent link="base_link"/>
+        <parent link="chassis"/>
         <child link="right_wheel"/>
-        <origin xyz="0 -0.3248 0.2032" rpy="${pi/2} 0 0" />
-        <axis xyz="0 0 -1"/>
+        <origin xyz="${-wheel_to_body_side} ${wheel_to_body_top} ${r_wheel}" rpy="0 0 0" />
+        <axis xyz="0 1 0"/>
+        <limit effort="50000" velocity="10"/>
+        <dynamic damping="1.0" friction="1.0"/>
     </joint>
     <link name="right_wheel">
         <visual>
-            <!-- <origin xyz="0 0.2032 0"/> -->
-            <geometry>
-                <cylinder radius="0.3048" length="0.04"/>
+            <origin xyz="0 0 0" rpy="${pi_const/2} 0 0"/>
+            <geometry>
+                <cylinder radius="${r_wheel}" length="${t_wheel}"/>
             </geometry>
             <material name="black"/>
         </visual>
         <collision>
-            <geometry>
-                <cylinder radius="0.3048" length="0.04"/>
-            </geometry>
-        </collision>
-        <xacro:inertial_cylinder mass="0.1" length="0.04" radius="0.3048">
-            <origin xyz="0 0 0" rpy="0 0 0"/>
-        </xacro:inertial_cylinder>
-    </link>
-    <gazebo reference="right_wheel">
-        <material>Gazebo/Black</material>
-    </gazebo>
+            <origin xyz="0 0 0" rpy="${pi_const/2} 0 0"/>
+            <geometry>
+                <cylinder radius="${r_wheel}" length="${t_wheel}"/>
+            </geometry>
+        </collision>
+        <xacro:inertia_wheel/>
+    </link>
     <!-- CASTER LEFT WHEEL LINK -->
     <joint name="caster_left_joint" type="continuous">
         <parent link="chassis"/>
         <child link="caster_left"/>
-        <origin xyz="1.1049 0.3148 0" rpy="${pi/2} 0 0" />
-        <axis xyz="0 0 -1"/>
+        <origin xyz="${caster_to_body_side} ${caster_to_body_top}  ${r_caster}" rpy="0 0 0" />
+        <axis xyz="0 1 0"/>
+        <limit effort="50000" velocity="10"/>
+        <dynamic damping="1.0" friction="1.0"/>
     </joint>
     <link name="caster_left">
         <visual>
-            <geometry>
-                <cylinder radius="0.1016" length="0.02"/>
-            </geometry>
-            <material name="black"/>
-        </visual>
-        <collision>
-            <geometry>
-                <cylinder radius="0.1016" length="0.2"/>
-            </geometry>
-        </collision>
-        <xacro:inertial_sphere mass="0.1" radius="0.1016">
-            <origin xyz="0 0 0" rpy="0 0 0"/>
-        </xacro:inertial_sphere>
-    </link>
-    <gazebo reference="caster_left">
-        <material>Gazebo/Black</material>
-        <!-- <mu1 value="0.001"/>
-        <mu2 value="0.001"/> -->
-    </gazebo>
+            <origin xyz="0 0 0" rpy="${pi_const/2} 0 0"/>
+            <geometry>
+                <cylinder radius="${r_caster}" length="${t_caster}"/>
+            </geometry>
+            <material name="blue"/>
+        </visual>
+        <collision>
+            <origin xyz="0 0 0" rpy="${pi_const/2} 0 0"/>
+            <geometry>
+                <cylinder radius="${r_caster}" length="${t_caster}"/>
+            </geometry>
+        </collision>
+        <xacro:inertia_caster/>
+    </link>
     <!-- CASTER RIGHT WHEEL LINK -->
     <joint name="caster_right_joint" type="continuous">
         <parent link="chassis"/>
         <child link="caster_right"/>
-        <origin xyz="1.1049 -0.3148 0" rpy="${pi/2} 0 0" />
-        <axis xyz="0 0 -1"/>
+        <origin xyz="${caster_to_body_side} ${-caster_to_body_top} ${r_caster}" rpy="0 0 0" />
+        <axis xyz="0 1 0"/>
+        <limit effort="50000" velocity="10"/>
+        <dynamic damping="1.0" friction="1.0"/>
     </joint>
     <link name="caster_right">
         <visual>
-            <geometry>
-                <cylinder radius="0.1016" length="0.02"/>
-            </geometry>
-            <material name="black"/>
-        </visual>
-        <collision>
-            <geometry>
-                <cylinder radius="0.1016" length="0.2"/>
-            </geometry>
-        </collision>
-        <xacro:inertial_sphere mass="0.1" radius="0.1016">
+            <origin xyz="0 0 0" rpy="${pi_const/2} 0 0"/>
+            <geometry>
+                <cylinder radius="${r_caster}" length="${t_caster}"/>
+            </geometry>
+            <material name="blue"/>
+        </visual>
+        <collision>
+            <origin xyz="0 0 0" rpy="${pi_const/2} 0 0"/>
+            <geometry>
+                <cylinder radius="${r_caster}" length="${t_caster}"/>
+            </geometry>
+        </collision>
+        <xacro:inertia_caster/>
+    </link>
+    <!-- ############################################################## -->
+    <!--                            LiDAR                               -->
+    <!-- ############################################################## -->
+    <joint name="lidar_joint" type="fixed">
+        <origin xyz="0 0 ${h+r_caster}" rpy="0 0 0"/>
+        <parent link="chassis"/>
+        <child link="lidar"/>
+        <axis xyz="0 1 0" rpy="0 0 0"/>
+    </joint>
+    <link name="lidar">
+        <visual>
+            <origin xyz="0 0 0.05" rpy="0 0 0"/>
+            <geometry>
+                <cylinder length="0.1" radius="0.1"/>
+            </geometry>
+        </visual>
+        <collision name='collision'>
+            <origin xyz="0 0 0.05" rpy="0 0 0"/>
+            <geometry>
+                <cylinder length="0.1" radius="0.1"/>
+            </geometry>
+        </collision>
+        <inertial>
+            <mass value="1e-6"/>
             <origin xyz="0 0 0" rpy="0 0 0"/>
-        </xacro:inertial_sphere>
-    </link>
-    <gazebo reference="caster_right">
-        <material>Gazebo/Black</material>
-        <!-- <mu1 value="0.001"/>
-        <mu2 value="0.001"/> -->
-    </gazebo>
+            <inertia ixx="1e-6" ixy="0" ixz="0"
+                     iyy="1e-6" iyz="0" izz="1e-6"/>
+        </inertial>
+    </link>
 </robot>
