Commit message: Setup gazebo simulation environment

File: description/robot_core.xacro (robot description, xacro)
@@ -42,7 +42,7 @@
         </xacro:inertial_box>
     </link>
-    <!-- <gazebo reference="chassis">
-        <material>Gazebo/White</material>
-    </gazebo> -->
+    <gazebo reference="chassis">
+        <material>Gazebo/Grey</material>
+    </gazebo>
     <!-- LEFT WHEEL LINK -->
     <joint name="left_wheel_joint" type="continuous">
@@ -69,7 +69,7 @@
         </xacro:inertial_cylinder>
     </link>
-    <!-- <gazebo reference="left_wheel">
-        <material>Gazebo/Blue</material>
-    </gazebo> -->
+    <gazebo reference="left_wheel">
+        <material>Gazebo/Black</material>
+    </gazebo>
     <!-- RIGHT WHEEL LINK -->
     <joint name="right_wheel_joint" type="continuous">
@@ -96,15 +96,15 @@
         </xacro:inertial_cylinder>
     </link>
-    <!-- <gazebo reference="right_wheel">
-        <material>Gazebo/Blue</material>
-    </gazebo> -->
+    <gazebo reference="right_wheel">
+        <material>Gazebo/Black</material>
+    </gazebo>
     <!-- CASTER LEFT WHEEL LINK -->
-    <joint name="caster_left_wheel_joint" type="continuous">
+    <joint name="caster_left_joint" type="continuous">
         <parent link="chassis"/>
-        <child link="caster_left_wheel"/>
+        <child link="caster_left"/>
         <origin xyz="1.1049 0.3148 0" rpy="${pi/2} 0 0" />
         <axis xyz="0 0 -1"/>
     </joint>
-    <link name="caster_left_wheel">
+    <link name="caster_left">
         <visual>
             <geometry>
@@ -122,17 +122,17 @@
         </xacro:inertial_sphere>
     </link>
-    <!-- <gazebo reference="caster_left_wheel">
+    <gazebo reference="caster_left">
         <material>Gazebo/Black</material>
-        <mu1 value="0.001"/>
-        <mu2 value="0.001"/>
-    </gazebo> -->
+        <!-- <mu1 value="0.001"/>
+        <mu2 value="0.001"/> -->
+    </gazebo>
     <!-- CASTER RIGHT WHEEL LINK -->
-    <joint name="caster_right_wheel_joint" type="continuous">
+    <joint name="caster_right_joint" type="continuous">
         <parent link="chassis"/>
-        <child link="caster_right_wheel"/>
+        <child link="caster_right"/>
         <origin xyz="1.1049 -0.3148 0" rpy="${pi/2} 0 0" />
         <axis xyz="0 0 -1"/>
     </joint>
-    <link name="caster_right_wheel">
+    <link name="caster_right">
         <visual>
             <geometry>
@@ -150,8 +150,8 @@
         </xacro:inertial_sphere>
     </link>
-    <!-- <gazebo reference="caster_wheel">
+    <gazebo reference="caster_right">
         <material>Gazebo/Black</material>
-        <mu1 value="0.001"/>
-        <mu2 value="0.001"/>
-    </gazebo> -->
+        <!-- <mu1 value="0.001"/>
+        <mu2 value="0.001"/> -->
+    </gazebo>
 </robot>
