Commit message: Setup gazebo to run with rviz for lidar simulation

File: description/robot_core.xacro (robot description, xacro)
@@ -164,5 +164,5 @@
         <parent link="chassis"/>
         <child link="caster_left"/>
-        <origin xyz="${caster_to_body_side} ${caster_to_body_top}  ${r_caster}" rpy="0 0 0" />
+        <origin xyz="${caster_to_body_side} ${-caster_to_body_top}  ${r_caster}" rpy="0 0 0" />
         <axis xyz="0 1 0"/>
         <limit effort="50000" velocity="10"/>
@@ -189,5 +189,5 @@
         <parent link="chassis"/>
         <child link="caster_right"/>
-        <origin xyz="${caster_to_body_side} ${-caster_to_body_top} ${r_caster}" rpy="0 0 0" />
+        <origin xyz="${caster_to_body_side} ${caster_to_body_top} ${r_caster}" rpy="0 0 0" />
         <axis xyz="0 1 0"/>
         <limit effort="50000" velocity="10"/>
@@ -225,4 +225,5 @@
                 <cylinder length="0.1" radius="0.1"/>
             </geometry>
+            <material name="red"/>
         </visual>
         <collision name='collision'>

Commit message: Added depth camera and SLAM toolbox ready

File: description/robot_core.xacro (robot description, xacro)
@@ -75,4 +75,7 @@
         <color rgba="0 0 1 1"/>
     </material>
+    <material name="red">
+        <color rgba="0 1 0 1"/>
+    </material>
     <material name="grey">
         <color rgba="1 1 1 1"/>
@@ -89,4 +92,11 @@
     <!-- Base Link-->
     <link name="base_link"></link>
+    <!-- Base_Footprint Link -->
+    <joint name="base_footprint_joint" type="fixed">
+        <parent link="base_link"/>
+        <child link="base_footprint"/>
+        <origin xyz="0 0 0" rpy="0 0 0"/>
+    </joint>
+    <link name="base_footprint"></link>
     <!-- Chassis-->
     <joint name="chassis_joint" type="fixed">
@@ -235,8 +245,41 @@
         <inertial>
             <mass value="1e-6"/>
-            <origin xyz="0 0 0" rpy="0 0 0"/>
+            <origin xyz="0 0 0.05" rpy="0 0 0"/>
             <inertia ixx="1e-6" ixy="0" ixz="0"
                      iyy="1e-6" iyz="0" izz="1e-6"/>
         </inertial>
     </link>
+    <!-- ############################################################## -->
+    <!--                         Depth Camera                           -->
+    <!-- ############################################################## -->
+    <joint name="camera_joint" type="fixed">
+        <parent link="chassis"/>
+        <child link="camera"/>
+        <origin xyz="0 0 ${h+r_caster+0.2}" rpy="0 0 0"/>
+    </joint>
+    <link name="camera">
+        <visual>
+            <geometry>
+                <box size="0.1 0.3 0.1"/>
+            </geometry>
+            <material name="black"/>
+        </visual>
+        <collision>
+            <geometry>
+                <box size="0.1 0.3 0.1"/>
+            </geometry>
+        </collision>
+        <inertial>
+            <mass value="0.1"/>
+            <origin xyz="0 0 0" rpy="0 0 0"/>
+            <inertia ixx="0.000166667" ixy="0" ixz="0"
+                     iyy="0.000166667" iyz="0" izz="0.000166667"/>
+        </inertial>
+    </link>
+    <joint name="camera_optical_joint" type="fixed">
+        <parent link="camera"/>
+        <child link="camera_optical"/>
+        <origin xyz="0 0 0" rpy="${-pi/2} 0 ${-pi/2}"/>
+    </joint>
+    <link name="camera_optical"/>
 </robot>

Commit message: Update depth camera and Gazebo bridge configuration

File: description/robot_core.xacro (robot description, xacro)
@@ -22,12 +22,8 @@
     <xacro:property name="wheel_to_body_top" value="${w/2+t_wheel/2}"/>
     <xacro:property name="caster_to_body_top" value="${w/2+t_caster/2}"/>
-    <!-- Material Density -->
-    <xacro:property name="d_body" value="7850.0"/>
-    <xacro:property name="d_wheel" value="7850.0"/>
-    <xacro:property name="d_caster" value="7850.0"/>
     <!-- Wheelchair Mass -->
-    <xacro:property name="m_body" value="${d_body*l*w*h}"/>
-    <xacro:property name="m_wheel" value="${d_wheel*pi_const*r_wheel*r_wheel*t_wheel}"/>
-    <xacro:property name="m_caster" value="${d_caster*pi_const*r_caster*r_caster*t_caster}"/>
+    <xacro:property name="m_body" value="20.0"/>
+    <xacro:property name="m_wheel" value="2.0"/>
+    <xacro:property name="m_caster" value="0.5"/>
     <!-- Moment of Inertia of Body -->
     <xacro:property name="Ix_body" value="${(1/12)*m_body*(h*h+w*w)}"/>
@@ -76,5 +72,5 @@
     </material>
     <material name="red">
-        <color rgba="0 1 0 1"/>
+        <color rgba="1 0 0 1"/>
     </material>
     <material name="grey">
@@ -124,5 +120,5 @@
         <parent link="chassis"/>
         <child link="left_wheel"/>
-        <origin xyz="${-wheel_to_body_side} ${-wheel_to_body_top} ${r_wheel}" rpy="0 0 0" />
+        <origin xyz="${-wheel_to_body_side} ${wheel_to_body_top} ${r_wheel}" rpy="0 0 0" />
         <axis xyz="0 1 0"/>
         <limit effort="50000" velocity="10"/>
@@ -149,5 +145,5 @@
         <parent link="chassis"/>
         <child link="right_wheel"/>
-        <origin xyz="${-wheel_to_body_side} ${wheel_to_body_top} ${r_wheel}" rpy="0 0 0" />
+        <origin xyz="${-wheel_to_body_side} ${-wheel_to_body_top} ${r_wheel}" rpy="0 0 0" />
         <axis xyz="0 1 0"/>
         <limit effort="50000" velocity="10"/>
@@ -226,8 +222,7 @@
         <origin xyz="0 0 ${h+r_caster}" rpy="0 0 0"/>
         <parent link="chassis"/>
-        <child link="lidar"/>
-        <axis xyz="0 1 0" rpy="0 0 0"/>
-    </joint>
-    <link name="lidar">
+        <child link="laser_frame"/>
+    </joint>
+    <link name="laser_frame">
         <visual>
             <origin xyz="0 0 0.05" rpy="0 0 0"/>
@@ -244,8 +239,8 @@
         </collision>
         <inertial>
-            <mass value="1e-6"/>
+            <mass value="0.2"/>
             <origin xyz="0 0 0.05" rpy="0 0 0"/>
-            <inertia ixx="1e-6" ixy="0" ixz="0"
-                     iyy="1e-6" iyz="0" izz="1e-6"/>
+            <inertia ixx="0.0006667" ixy="0" ixz="0"
+                     iyy="0.0006667" iyz="0" izz="0.001"/>
         </inertial>
     </link>
@@ -255,8 +250,8 @@
     <joint name="camera_joint" type="fixed">
         <parent link="chassis"/>
-        <child link="camera"/>
+        <child link="camera_link"/>
         <origin xyz="0 0 ${h+r_caster+0.2}" rpy="0 0 0"/>
     </joint>
-    <link name="camera">
+    <link name="camera_link">
         <visual>
             <geometry>
@@ -273,13 +268,13 @@
             <mass value="0.1"/>
             <origin xyz="0 0 0" rpy="0 0 0"/>
-            <inertia ixx="0.000166667" ixy="0" ixz="0"
-                     iyy="0.000166667" iyz="0" izz="0.000166667"/>
+            <inertia ixx="0.000833333" ixy="0" ixz="0"
+                     iyy="0.000166667" iyz="0" izz="0.000833333"/>
         </inertial>
     </link>
     <joint name="camera_optical_joint" type="fixed">
-        <parent link="camera"/>
-        <child link="camera_optical"/>
+        <parent link="camera_link"/>
+        <child link="camera_link_optical"/>
         <origin xyz="0 0 0" rpy="${-pi/2} 0 ${-pi/2}"/>
     </joint>
-    <link name="camera_optical"/>
+    <link name="camera_link_optical"/>
 </robot>

File: description/robot_core_test.xacro (robot description, xacro)
@@ -7,43 +7,43 @@
     <xacro:property name="pi_const" value="3.14159265" />
     <!-- Body Dimensions -->
-    <xacro:property name="a" value="1.0"/>
-    <xacro:property name="b" value="0.3"/>
-    <xacro:property name="c" value="0.6"/>
+    <xacro:property name="l" value="1.1049"/>
+    <xacro:property name="w" value="0.6096"/>
+    <xacro:property name="h" value="0.6144"/>   <!-- actual: 0.9144-->
     <!-- Wheel Dimension -->
-    <xacro:property name="r" value="0.15"/>
-    <xacro:property name="d" value="0.1"/>
+    <xacro:property name="r_wheel" value="0.3048"/>
+    <xacro:property name="t_wheel" value="0.0400"/>
     <!-- Caster Dimension -->
-    <!-- <xacro:property name="r_caster" value="0.1016"/>
-    <xacro:property name="t_caster" value="0.0200"/> -->
+    <xacro:property name="r_caster" value="0.1016"/>
+    <xacro:property name="t_caster" value="0.0200"/>
     <!-- Distance btw Centers -->
-    <xacro:property name="s1" value="${b/2+r}"/>
-    <xacro:property name="s2" value="${2*r}"/>
-    <xacro:property name="s3" value="${2*r}"/>
-    <xacro:property name="s4" value="${c/2+d/2}"/>
-    <!-- <xacro:property name="caster_to_body_top" value="${w/2+t_caster/2}"/> -->
+    <xacro:property name="body_to_gnd" value="${h/2+r_caster}"/>
+    <xacro:property name="wheel_to_body_side" value="0.55245"/>
+    <xacro:property name="caster_to_body_side" value="0.14605"/>
+    <xacro:property name="wheel_to_body_top" value="${w/2+t_wheel/2}"/>
+    <xacro:property name="caster_to_body_top" value="${w/2+t_caster/2}"/>
     <!-- Material Density -->
-    <xacro:property name="d1" value="2710.0"/>
-    <xacro:property name="d2" value="2710.0"/>
-    <xacro:property name="d3" value="2710.0"/>
+    <xacro:property name="d_body" value="7850.0"/>
+    <xacro:property name="d_wheel" value="7850.0"/>
+    <xacro:property name="d_caster" value="7850.0"/>
     <!-- Wheelchair Mass -->
-    <xacro:property name="m1" value="${d1*a*c*b}"/>
-    <xacro:property name="m2" value="${d2*pi_const*r*r*d}"/>
-    <xacro:property name="m3" value="${d3*(4.0/3.0)*pi_const*r*r*r}"/>
+    <xacro:property name="m_body" value="${d_body*l*w*h}"/>
+    <xacro:property name="m_wheel" value="${d_wheel*pi_const*r_wheel*r_wheel*t_wheel}"/>
+    <xacro:property name="m_caster" value="${d_caster*pi_const*r_caster*r_caster*t_caster}"/>
     <!-- Moment of Inertia of Body -->
-    <xacro:property name="Ix_body" value="${(1/12)*m1*(b*b+c*c)}"/>
-    <xacro:property name="Iy_body" value="${(1/12)*m1*(a*a+b*b)}"/>
-    <xacro:property name="Iz_body" value="${(1/12)*m1*(a*a+c*c)}"/>
+    <xacro:property name="Ix_body" value="${(1/12)*m_body*(h*h+w*w)}"/>
+    <xacro:property name="Iy_body" value="${(1/12)*m_body*(l*l+h*h)}"/>
+    <xacro:property name="Iz_body" value="${(1/12)*m_body*(l*l+w*w)}"/>
     <!-- Moment of Inertia of Wheel -->
-    <xacro:property name="I_wheel" value="${(1.0/12.0)*m2*(3.0*r*r+d*d)}"/>
-    <xacro:property name="Iz_wheel" value="${0.5*m2*r*r}"/>
+    <xacro:property name="I_wheel" value="${(1.0/12.0)*m_wheel*(3.0*r_wheel*r_wheel+t_wheel*t_wheel)}"/>
+    <xacro:property name="Iz_wheel" value="${0.5*m_wheel*r_wheel*r_wheel}"/>
     <!-- Moment of Inertia of Caster -->
-    <xacro:property name="I_caster" value="${(2.0/5.0)*m3*r*r}"/>
-    <!-- <xacro:property name="Iz_caster" value="${0.5*m_caster*r_caster*r_caster}"/> -->
+    <xacro:property name="I_caster" value="${(1.0/12.0)*m_caster*(3.0*r_caster*r_caster+t_caster*t_caster)}"/>
+    <xacro:property name="Iz_caster" value="${0.5*m_caster*r_caster*r_caster}"/>
     <!-- Macro for Inertial Section -->
     <xacro:macro name="inertia_body">
         <!-- displacement & rientation of center of mass frame of link to ground -->
         <inertial>
-            <origin xyz="0 0 ${s1}" rpy="0 0 0"/>
-            <mass value="${m1}"/>
+            <origin xyz="0 0 ${body_to_gnd}" rpy="0 0 0"/>
+            <mass value="${m_body}"/>
             <inertia ixx="${Ix_body}" ixy="0.0" ixz="0.0"
                      iyy="${Iy_body}" iyz="0.0"
@@ -53,6 +53,6 @@
     <xacro:macro name="inertia_wheel">
         <inertial>
-            <origin xyz="0 0 0" rpy="1.570795 0 0"/>
-            <mass value="${m2}"/>
+            <origin xyz="0 0 0" rpy="${pi_const/2} 0 0"/>
+            <mass value="${m_wheel}"/>
             <inertia ixx="${I_wheel}" ixy="0.0" ixz="0.0"
                      iyy="${I_wheel}" iyz="0.0"
@@ -62,13 +62,13 @@
     <xacro:macro name="inertia_caster">
         <inertial>
-            <origin xyz="0 0 0" rpy="0 0 0"/>
-            <mass value="${m3}"/>
+            <origin xyz="0 0 0" rpy="${pi_const/2} 0 0"/>
+            <mass value="${m_caster}"/>
             <inertia ixx="${I_caster}" ixy="0.0" ixz="0.0"
                      iyy="${I_caster}" iyz="0.0"
-                     izz="${I_caster}"/>
+                     izz="${Iz_caster}"/>
         </inertial>
     </xacro:macro>
     <!-- Additional Files -->
-    <xacro:include filename="$(find wheelchair_one)/description/gazebo_control_test"/>
+    <xacro:include filename="$(find wheelchair_one)/description/gazebo_control"/>
     <!-- colors -->
     <material name="blue">
@@ -91,34 +91,29 @@
     <!-- ############################################################## -->
     <!-- Base Link-->
-    <joint name="base_link_joint" type="fixed">
-        <parent link="base_link"/>
-        <child link="chassis"/>
-        <origin xyz="0 0 0" rpy="0 0 0"/>
-    </joint>
     <link name="base_link"></link>
     <!-- Base_Footprint Link -->
-    <!-- <joint name="base_footprint_joint" type="fixed">
+    <joint name="base_footprint_joint" type="fixed">
         <parent link="base_link"/>
         <child link="base_footprint"/>
         <origin xyz="0 0 0" rpy="0 0 0"/>
     </joint>
-    <link name="base_footprint"></link> -->
+    <link name="base_footprint"></link>
     <!-- Chassis-->
-    <!-- <joint name="chassis_joint" type="fixed">
+    <joint name="chassis_joint" type="fixed">
         <parent link="base_link"/>
         <child link="chassis"/>
-    </joint> -->
+    </joint>
     <link name="chassis">
         <visual>
-            <origin xyz="0 0 ${s1}" rpy="0 0 0"/>
-            <geometry>
-                <box size="${a} ${c} ${b}"/>
+            <origin xyz="0 0 ${body_to_gnd}" rpy="0 0 0"/>
+            <geometry>
+                <box size="${l} ${w} ${h}"/>
             </geometry>
             <material name="grey"/>
         </visual>
         <collision>
-            <origin xyz="0 0 ${s1}" rpy="0 0 0"/>
-            <geometry>
-                <box size="${a} ${c} ${b}"/>
+            <origin xyz="0 0 ${body_to_gnd}" rpy="0 0 0"/>
+            <geometry>
+                <box size="${l} ${w} ${h}"/>
             </geometry>
         </collision>
@@ -129,5 +124,5 @@
         <parent link="chassis"/>
         <child link="left_wheel"/>
-        <origin xyz="${-s2} ${-s4} ${r}" rpy="0 0 0" />
+        <origin xyz="${-wheel_to_body_side} ${-wheel_to_body_top} ${r_wheel}" rpy="0 0 0" />
         <axis xyz="0 1 0"/>
         <limit effort="50000" velocity="10"/>
@@ -136,14 +131,14 @@
     <link name="left_wheel">
         <visual>
-            <origin xyz="0 0 0" rpy="1.570795 0 0"/>
-            <geometry>
-                <cylinder radius="${r}" length="${d}"/>
+            <origin xyz="0 0 0" rpy="${pi_const/2} 0 0"/>
+            <geometry>
+                <cylinder radius="${r_wheel}" length="${t_wheel}"/>
             </geometry>
             <material name="black"/>
         </visual>
         <collision>
-            <origin xyz="0 0 0" rpy="1.570795 0 0"/>
-            <geometry>
-                <cylinder radius="${r}" length="${d}"/>
+            <origin xyz="0 0 0" rpy="${pi_const/2} 0 0"/>
+            <geometry>
+                <cylinder radius="${r_wheel}" length="${t_wheel}"/>
             </geometry>
         </collision>
@@ -154,5 +149,5 @@
         <parent link="chassis"/>
         <child link="right_wheel"/>
-        <origin xyz="${-s2} ${s4} ${r}" rpy="0 0 0" />
+        <origin xyz="${-wheel_to_body_side} ${wheel_to_body_top} ${r_wheel}" rpy="0 0 0" />
         <axis xyz="0 1 0"/>
         <limit effort="50000" velocity="10"/>
@@ -161,36 +156,39 @@
     <link name="right_wheel">
         <visual>
-            <origin xyz="0 0 0" rpy="1.570795 0 0"/>
-            <geometry>
-                <cylinder radius="${r}" length="${d}"/>
+            <origin xyz="0 0 0" rpy="${pi_const/2} 0 0"/>
+            <geometry>
+                <cylinder radius="${r_wheel}" length="${t_wheel}"/>
             </geometry>
             <material name="black"/>
         </visual>
         <collision>
-            <origin xyz="0 0 0" rpy="1.570795 0 0"/>
-            <geometry>
-                <cylinder radius="${r}" length="${d}"/>
+            <origin xyz="0 0 0" rpy="${pi_const/2} 0 0"/>
+            <geometry>
+                <cylinder radius="${r_wheel}" length="${t_wheel}"/>
             </geometry>
         </collision>
         <xacro:inertia_wheel/>
     </link>
-    <!-- CASTER WHEEL LINK -->
-    <joint name="caster_joint" type="continuous">
-        <parent link="chassis"/>
-        <child link="caster"/>
-        <origin xyz="${s3} 0 ${r}" rpy="0 0 0" />
-    </joint>
-    <link name="caster">
-        <visual>
-            <origin xyz="0 0 0" rpy="0 0 0"/>
-            <geometry>
-                <sphere radius="${r}"/>
+    <!-- CASTER LEFT WHEEL LINK -->
+    <joint name="caster_left_joint" type="continuous">
+        <parent link="chassis"/>
+        <child link="caster_left"/>
+        <origin xyz="${caster_to_body_side} ${-caster_to_body_top}  ${r_caster}" rpy="0 0 0" />
+        <axis xyz="0 1 0"/>
+        <limit effort="50000" velocity="10"/>
+        <dynamic damping="1.0" friction="1.0"/>
+    </joint>
+    <link name="caster_left">
+        <visual>
+            <origin xyz="0 0 0" rpy="${pi_const/2} 0 0"/>
+            <geometry>
+                <cylinder radius="${r_caster}" length="${t_caster}"/>
             </geometry>
             <material name="blue"/>
         </visual>
         <collision>
-            <origin xyz="0 0 0" rpy="0 0 0"/>
-            <geometry>
-                <sphere radius="${r}"/>
+            <origin xyz="0 0 0" rpy="${pi_const/2} 0 0"/>
+            <geometry>
+                <cylinder radius="${r_caster}" length="${t_caster}"/>
             </geometry>
         </collision>
@@ -198,5 +196,5 @@
     </link>
     <!-- CASTER RIGHT WHEEL LINK -->
-    <!-- <joint name="caster_right_joint" type="continuous">
+    <joint name="caster_right_joint" type="continuous">
         <parent link="chassis"/>
         <child link="caster_right"/>
@@ -221,15 +219,14 @@
         </collision>
         <xacro:inertia_caster/>
-    </link> -->
+    </link>
     <!-- ############################################################## -->
     <!--                            LiDAR                               -->
     <!-- ############################################################## -->
-    <joint name="lidar_joint" type="fixed">
-        <origin xyz="0 0 ${b+r}" rpy="0 0 0"/>
-        <parent link="chassis"/>
-        <child link="lidar"/>
-        <axis xyz="0 1 0"/>
-    </joint>
-    <link name="lidar">
+    <joint name="laser_joint" type="fixed">
+        <origin xyz="0 0 ${h+r_caster}" rpy="0 0 0"/>
+        <parent link="chassis"/>
+        <child link="laser_frame"/>
+    </joint>
+    <link name="laser_frame">
         <visual>
             <origin xyz="0 0 0.05" rpy="0 0 0"/>
@@ -247,5 +244,5 @@
         <inertial>
             <mass value="1e-6"/>
-            <origin xyz="0 0 0" rpy="0 0 0"/>
+            <origin xyz="0 0 0.05" rpy="0 0 0"/>
             <inertia ixx="1e-6" ixy="0" ixz="0"
                      iyy="1e-6" iyz="0" izz="1e-6"/>
@@ -257,8 +254,8 @@
     <joint name="camera_joint" type="fixed">
         <parent link="chassis"/>
-        <child link="camera"/>
-        <origin xyz="0 0 ${b+r+0.2}" rpy="0 0 0"/>
-    </joint>
-    <link name="camera">
+        <child link="camera_link"/>
+        <origin xyz="0 0 ${h+r_caster+0.2}" rpy="0 0 0"/>
+    </joint>
+    <link name="camera_link">
         <visual>
             <geometry>
@@ -280,8 +277,8 @@
     </link>
     <joint name="camera_optical_joint" type="fixed">
-        <parent link="camera"/>
-        <child link="camera_optical"/>
+        <parent link="camera_link"/>
+        <child link="camera_link_optical"/>
         <origin xyz="0 0 0" rpy="${-pi/2} 0 ${-pi/2}"/>
     </joint>
-    <link name="camera_optical"/>
+    <link name="camera_link_optical"/>
 </robot>
