Commit message: Testing with physical lidar

File: description/robot_core1.xacro (robot description, xacro)
@@ -91,17 +91,17 @@
     <!-- ############################################################## -->
     <!-- Base Link-->
-    <joint name="base_link_joint" type="fixed">
+    <!-- <joint name="base_link_joint" type="fixed">
         <parent link="base_link"/>
-        <child link="chassis"/>
+        <child link="base_footprint"/>
         <origin xyz="0 0 0" rpy="0 0 0"/>
-    </joint>
+    </joint> -->
     <link name="base_link"></link>
     <!-- Base_Footprint Link -->
-    <!-- <joint name="base_footprint_joint" type="fixed">
+    <joint name="base_footprint_joint" type="fixed">
         <parent link="base_link"/>
         <child link="base_footprint"/>
         <origin xyz="0 0 0" rpy="0 0 0"/>
     </joint>
-    <link name="base_footprint"></link> -->
+    <link name="base_footprint"></link>
     <!-- Chassis-->
     <!-- <joint name="chassis_joint" type="fixed">
@@ -109,132 +109,16 @@
         <child link="chassis"/>
     </joint> -->
-    <link name="chassis">
-        <visual>
-            <origin xyz="0 0 ${body_to_gnd}" rpy="0 0 0"/>
-            <geometry>
-                <box size="${l} ${w} ${h}"/>
-            </geometry>
-            <material name="grey"/>
-        </visual>
-        <collision>
-            <origin xyz="0 0 ${body_to_gnd}" rpy="0 0 0"/>
-            <geometry>
-                <box size="${l} ${w} ${h}"/>
-            </geometry>
-        </collision>
-        <xacro:inertia_body/>
-    </link>
-    <!-- LEFT WHEEL LINK -->
-    <joint name="left_wheel_joint" type="continuous">
-        <parent link="chassis"/>
-        <child link="left_wheel"/>
-        <origin xyz="${-wheel_to_body_side} ${-wheel_to_body_top} ${r_wheel}" rpy="0 0 0" />
-        <axis xyz="0 1 0"/>
-        <limit effort="50000" velocity="10"/>
-        <dynamic damping="1.0" friction="1.0"/>
-    </joint>
-    <link name="left_wheel">
-        <visual>
-            <origin xyz="0 0 0" rpy="${pi_const/2} 0 0"/>
-            <geometry>
-                <cylinder radius="${r_wheel}" length="${t_wheel}"/>
-            </geometry>
-            <material name="black"/>
-        </visual>
-        <collision>
-            <origin xyz="0 0 0" rpy="${pi_const/2} 0 0"/>
-            <geometry>
-                <cylinder radius="${r_wheel}" length="${t_wheel}"/>
-            </geometry>
-        </collision>
-        <xacro:inertia_wheel/>
-    </link>
-    <!-- RIGHT WHEEL LINK -->
-    <joint name="right_wheel_joint" type="continuous">
-        <parent link="chassis"/>
-        <child link="right_wheel"/>
-        <origin xyz="${-wheel_to_body_side} ${wheel_to_body_top} ${r_wheel}" rpy="0 0 0" />
-        <axis xyz="0 1 0"/>
-        <limit effort="50000" velocity="10"/>
-        <dynamic damping="1.0" friction="1.0"/>
-    </joint>
-    <link name="right_wheel">
-        <visual>
-            <origin xyz="0 0 0" rpy="${pi_const/2} 0 0"/>
-            <geometry>
-                <cylinder radius="${r_wheel}" length="${t_wheel}"/>
-            </geometry>
-            <material name="black"/>
-        </visual>
-        <collision>
-            <origin xyz="0 0 0" rpy="${pi_const/2} 0 0"/>
-            <geometry>
-                <cylinder radius="${r_wheel}" length="${t_wheel}"/>
-            </geometry>
-        </collision>
-        <xacro:inertia_wheel/>
-    </link>
-    <!-- CASTER LEFT WHEEL LINK -->
-    <joint name="caster_left_joint" type="continuous">
-        <parent link="chassis"/>
-        <child link="caster_left"/>
-        <origin xyz="${caster_to_body_side} ${-caster_to_body_top}  ${r_caster}" rpy="0 0 0" />
-        <axis xyz="0 1 0"/>
-        <limit effort="50000" velocity="10"/>
-        <dynamic damping="1.0" friction="1.0"/>
-    </joint>
-    <link name="caster_left">
-        <visual>
-            <origin xyz="0 0 0" rpy="${pi_const/2} 0 0"/>
-            <geometry>
-                <cylinder radius="${r_caster}" length="${t_caster}"/>
-            </geometry>
-            <material name="blue"/>
-        </visual>
-        <collision>
-            <origin xyz="0 0 0" rpy="${pi_const/2} 0 0"/>
-            <geometry>
-                <cylinder radius="${r_caster}" length="${t_caster}"/>
-            </geometry>
-        </collision>
-        <xacro:inertia_caster/>
-    </link>
-    <!-- CASTER RIGHT WHEEL LINK -->
-    <joint name="caster_right_joint" type="continuous">
-        <parent link="chassis"/>
-        <child link="caster_right"/>
-        <origin xyz="${caster_to_body_side} ${caster_to_body_top} ${r_caster}" rpy="0 0 0" />
-        <axis xyz="0 1 0"/>
-        <limit effort="50000" velocity="10"/>
-        <dynamic damping="1.0" friction="1.0"/>
-    </joint>
-    <link name="caster_right">
-        <visual>
-            <origin xyz="0 0 0" rpy="${pi_const/2} 0 0"/>
-            <geometry>
-                <cylinder radius="${r_caster}" length="${t_caster}"/>
-            </geometry>
-            <material name="blue"/>
-        </visual>
-        <collision>
-            <origin xyz="0 0 0" rpy="${pi_const/2} 0 0"/>
-            <geometry>
-                <cylinder radius="${r_caster}" length="${t_caster}"/>
-            </geometry>
-        </collision>
-        <xacro:inertia_caster/>
-    </link>
     <!-- ############################################################## -->
     <!--                            LiDAR                               -->
     <!-- ############################################################## -->
     <joint name="lidar_joint" type="fixed">
-        <origin xyz="0 0 ${h+r_caster}" rpy="0 0 0"/>
-        <parent link="chassis"/>
-        <child link="lidar"/>
+        <origin xyz="0 0 0.18" rpy="0 0 0"/>
+        <parent link="base_footprint"/>
+        <child link="base_laser"/>
         <axis xyz="0 1 0" rpy="0 0 0"/>
     </joint>
-    <link name="lidar">
+    <link name="base_laser">
         <visual>
-            <origin xyz="0 0 0.05" rpy="0 0 0"/>
+            <origin xyz="0 0 0.1" rpy="0 0 0"/>
             <geometry>
                 <cylinder length="0.1" radius="0.1"/>
@@ -243,5 +127,5 @@
         </visual>
         <collision name='collision'>
-            <origin xyz="0 0 0.05" rpy="0 0 0"/>
+            <origin xyz="0 0 0.1" rpy="0 0 0"/>
             <geometry>
                 <cylinder length="0.1" radius="0.1"/>
@@ -250,5 +134,5 @@
         <inertial>
             <mass value="1e-6"/>
-            <origin xyz="0 0 0.05" rpy="0 0 0"/>
+            <origin xyz="0 0 0.1" rpy="0 0 0"/>
             <inertia ixx="1e-6" ixy="0" ixz="0"
                      iyy="1e-6" iyz="0" izz="1e-6"/>
@@ -258,5 +142,5 @@
     <!--                         Depth Camera                           -->
     <!-- ############################################################## -->
-    <joint name="camera_joint" type="fixed">
+    <!-- <joint name="camera_joint" type="fixed">
         <parent link="chassis"/>
         <child link="camera"/>
@@ -287,4 +171,4 @@
         <origin xyz="0 0 0" rpy="${-pi/2} 0 ${-pi/2}"/>
     </joint>
-    <link name="camera_optical"/>
+    <link name="camera_optical"/> -->
 </robot>
